Commit message: Update robot_core.xacro

File: articubot_one/description/robot_core.xacro (robot description, xacro)
@@ -126,5 +126,5 @@
             </geometry>
         </collision>
-        <xacro:inertial_cylinder mass="0.2" length="0.15" radius="0.18">
+        <xacro:inertial_cylinder mass="0.1" length="0.15" radius="0.18">
             <origin xyz="0 0 -0.025" rpy="0 0 ${pi/2}"/>
         </xacro:inertial_cylinder>
@@ -150,5 +150,5 @@
             </geometry>
         </collision>
-        <xacro:inertial_cylinder mass="0.2" length="0.15" radius="0.18">
+        <xacro:inertial_cylinder mass="0.1" length="0.15" radius="0.18">
             <origin xyz="0 0 -0.025" rpy="0 0 ${pi/2}"/>
         </xacro:inertial_cylinder>
@@ -175,5 +175,5 @@
             </geometry>
         </collision>
-        <xacro:inertial_cylinder mass="0.01" length="0.65" radius="0.03">
+        <xacro:inertial_cylinder mass="0.1" length="0.65" radius="0.03">
             <origin xyz="0 0 0.35" rpy="0 0 0"/>
         </xacro:inertial_cylinder>
@@ -200,5 +200,5 @@
             </geometry>
         </collision>
-        <xacro:inertial_cylinder mass="0.025" length="0.65" radius="0.03">
+        <xacro:inertial_cylinder mass="0.1" length="0.65" radius="0.03">
             <origin xyz="0 0 0.35" rpy="0 0 0"/>
         </xacro:inertial_cylinder>
@@ -225,5 +225,5 @@
             </geometry>
         </collision>
-        <xacro:inertial_cylinder mass="0.025" length="0.3" radius="0.03">
+        <xacro:inertial_cylinder mass="0.05" length="0.3" radius="0.03">
             <origin xyz="0 -0.2 0.05 " rpy="${pi/1.9} 0 0"/>
         </xacro:inertial_cylinder>
@@ -250,16 +250,16 @@
             </geometry>
         </collision>
-        <xacro:inertial_cylinder mass="0.01" length="0.3" radius="0.03">
+        <xacro:inertial_cylinder mass="0.05" length="0.3" radius="0.03">
             <origin xyz="0 -0.2 0.05 " rpy="${pi/1.9} 0 0"/>
         </xacro:inertial_cylinder>
     </link>
     <!-- Loader -->
-    <joint name="Loader_joint" type="continuous">
+    <joint name="Loader_joint" type="revolute">
         <parent link="Left_Curve"/>
         <child link="Loader"/>
-        <origin xyz="-0.25 -0.4 -0.018" rpy="${pi/6} 0 0"/>
+        <origin xyz="-0.24 -0.4 -0.018" rpy="${pi/5} 0 0"/>
         <axis xyz="1 0 0"/>
         <dynamics friction="1"/>
-        <!-- <limit lower="0" upper="-0.82" velocity="0.1" effort="100" /> -->
+        <limit lower="-0.1" upper="-0.82" velocity="0.1" effort="100" />
     </joint>
     <link name="Loader">
@@ -275,6 +275,6 @@
             </geometry>
         </collision>
-        <xacro:inertial_box mass="0.05" x="0.6" y="0.2" z="0.3">
-            <origin xyz="-0.2 -0.12 0.14" rpy="0 0 0"/>
+        <xacro:inertial_box mass="0.05" x="0.6" y="0.02" z="0.4">
+            <origin xyz="0 -0.2 0.14" rpy="0 0 0"/>
         </xacro:inertial_box>
     </link>
